Commit message: Update robot description and check mesh origin script

File: Robot_description/urdf/Robot.xacro (robot description, xacro)
@@ -31,5 +31,5 @@
   </inertial>
   <visual>
-    <origin xyz="0.0644 -0.00785 -0.041328" rpy="0 0 0"/>
+    <origin xyz="0 0 0" rpy="0 0 0"/>
     <geometry>
       <mesh filename="file://$(find Robot_description)/meshes/Dynamixel_AX12a_1.stl" scale="0.001 0.001 0.001"/>
@@ -38,5 +38,5 @@
   </visual>
   <collision>
-    <origin xyz="0.0644 -0.00785 -0.041328" rpy="0 0 0"/>
+    <origin xyz="0 0 0" rpy="0 0 0"/>
     <geometry>
       <mesh filename="file://$(find Robot_description)/meshes/Dynamixel_AX12a_1.stl" scale="0.001 0.001 0.001"/>
@@ -51,5 +51,5 @@
   </inertial>
   <visual>
-    <origin xyz="0.0972 -0.03785 0.041328" rpy="0 0 0"/>
+    <origin xyz="0 0 0" rpy="0 0 0"/>
     <geometry>
       <mesh filename="file://$(find Robot_description)/meshes/Dynamixel_AX12a__1__1.stl" scale="0.001 0.001 0.001"/>
@@ -58,5 +58,5 @@
   </visual>
   <collision>
-    <origin xyz="0.0972 -0.03785 0.041328" rpy="0 0 0"/>
+    <origin xyz="0 0 0" rpy="0 0 0"/>
     <geometry>
       <mesh filename="file://$(find Robot_description)/meshes/Dynamixel_AX12a__1__1.stl" scale="0.001 0.001 0.001"/>
@@ -71,5 +71,5 @@
   </inertial>
   <visual>
-    <origin xyz="-0.0972 -0.00785 -0.041328" rpy="0 0 0"/>
+    <origin xyz="0 0 0" rpy="0 0 0"/>
     <geometry>
       <mesh filename="file://$(find Robot_description)/meshes/Dynamixel_AX12a__2__1.stl" scale="0.001 0.001 0.001"/>
@@ -78,5 +78,5 @@
   </visual>
   <collision>
-    <origin xyz="-0.0972 -0.00785 -0.041328" rpy="0 0 0"/>
+    <origin xyz="0 0 0" rpy="0 0 0"/>
     <geometry>
       <mesh filename="file://$(find Robot_description)/meshes/Dynamixel_AX12a__2__1.stl" scale="0.001 0.001 0.001"/>
@@ -91,5 +91,5 @@
   </inertial>
   <visual>
-    <origin xyz="-0.0972 -0.00785 0.041328" rpy="0 0 0"/>
+    <origin xyz="0 0 0" rpy="0 0 0"/>
     <geometry>
       <mesh filename="file://$(find Robot_description)/meshes/Dynamixel_AX12a__3__1.stl" scale="0.001 0.001 0.001"/>
@@ -98,5 +98,5 @@
   </visual>
   <collision>
-    <origin xyz="-0.0972 -0.00785 0.041328" rpy="0 0 0"/>
+    <origin xyz="0 0 0" rpy="0 0 0"/>
     <geometry>
       <mesh filename="file://$(find Robot_description)/meshes/Dynamixel_AX12a__3__1.stl" scale="0.001 0.001 0.001"/>
@@ -111,5 +111,5 @@
   </inertial>
   <visual>
-    <origin xyz="0.062842 -0.036345 -0.153336" rpy="0 0 0"/>
+    <origin xyz="0 0 0" rpy="0 0 0"/>
     <geometry>
       <mesh filename="file://$(find Robot_description)/meshes/Robot_Dog_femur__3__1.stl" scale="0.001 0.001 0.001"/>
@@ -118,5 +118,5 @@
   </visual>
   <collision>
-    <origin xyz="0.062842 -0.036345 -0.153336" rpy="0 0 0"/>
+    <origin xyz="0 0 0" rpy="0 0 0"/>
     <geometry>
       <mesh filename="file://$(find Robot_description)/meshes/Robot_Dog_femur__3__1.stl" scale="0.001 0.001 0.001"/>
@@ -131,5 +131,5 @@
   </inertial>
   <visual>
-    <origin xyz="-0.098802 -0.036645 -0.153336" rpy="0 0 0"/>
+    <origin xyz="0 0 0" rpy="0 0 0"/>
     <geometry>
       <mesh filename="file://$(find Robot_description)/meshes/Robot_Dog_femur_1.stl" scale="0.001 0.001 0.001"/>
@@ -138,5 +138,5 @@
   </visual>
   <collision>
-    <origin xyz="-0.098802 -0.036645 -0.153336" rpy="0 0 0"/>
+    <origin xyz="0 0 0" rpy="0 0 0"/>
     <geometry>
       <mesh filename="file://$(find Robot_description)/meshes/Robot_Dog_femur_1.stl" scale="0.001 0.001 0.001"/>
@@ -151,5 +151,5 @@
   </inertial>
   <visual>
-    <origin xyz="0.06285 -0.036345 0.153336" rpy="0 0 0"/>
+    <origin xyz="0 0 0" rpy="0 0 0"/>
     <geometry>
       <mesh filename="file://$(find Robot_description)/meshes/Robot_Dog_femur__2__1.stl" scale="0.001 0.001 0.001"/>
@@ -158,5 +158,5 @@
   </visual>
   <collision>
-    <origin xyz="0.06285 -0.036345 0.153336" rpy="0 0 0"/>
+    <origin xyz="0 0 0" rpy="0 0 0"/>
     <geometry>
       <mesh filename="file://$(find Robot_description)/meshes/Robot_Dog_femur__2__1.stl" scale="0.001 0.001 0.001"/>
@@ -171,5 +171,5 @@
   </inertial>
   <visual>
-    <origin xyz="-0.098442 -0.036245 0.153336" rpy="0 0 0"/>
+    <origin xyz="0 0 0" rpy="0 0 0"/>
     <geometry>
       <mesh filename="file://$(find Robot_description)/meshes/Robot_Dog_femur__1__1.stl" scale="0.001 0.001 0.001"/>
@@ -178,5 +178,5 @@
   </visual>
   <collision>
-    <origin xyz="-0.098442 -0.036245 0.153336" rpy="0 0 0"/>
+    <origin xyz="0 0 0" rpy="0 0 0"/>
     <geometry>
       <mesh filename="file://$(find Robot_description)/meshes/Robot_Dog_femur__1__1.stl" scale="0.001 0.001 0.001"/>
@@ -191,5 +191,5 @@
   </inertial>
   <visual>
-    <origin xyz="0.007952 0.058574 0.155336" rpy="0 0 0"/>
+    <origin xyz="0 0 0" rpy="0 0 0"/>
     <geometry>
       <mesh filename="file://$(find Robot_description)/meshes/Robot_Dog_TIBIA_1.stl" scale="0.001 0.001 0.001"/>
@@ -198,5 +198,5 @@
   </visual>
   <collision>
-    <origin xyz="0.007952 0.058574 0.155336" rpy="0 0 0"/>
+    <origin xyz="0 0 0" rpy="0 0 0"/>
     <geometry>
       <mesh filename="file://$(find Robot_description)/meshes/Robot_Dog_TIBIA_1.stl" scale="0.001 0.001 0.001"/>
@@ -211,5 +211,5 @@
   </inertial>
   <visual>
-    <origin xyz="-0.15334 0.058674 0.155336" rpy="0 0 0"/>
+    <origin xyz="0 0 0" rpy="0 0 0"/>
     <geometry>
       <mesh filename="file://$(find Robot_description)/meshes/Robot_Dog_TIBIA__1__1.stl" scale="0.001 0.001 0.001"/>
@@ -218,5 +218,5 @@
   </visual>
   <collision>
-    <origin xyz="-0.15334 0.058674 0.155336" rpy="0 0 0"/>
+    <origin xyz="0 0 0" rpy="0 0 0"/>
     <geometry>
       <mesh filename="file://$(find Robot_description)/meshes/Robot_Dog_TIBIA__1__1.stl" scale="0.001 0.001 0.001"/>
@@ -231,5 +231,5 @@
   </inertial>
   <visual>
-    <origin xyz="0.008089 0.058658 -0.155336" rpy="0 0 0"/>
+    <origin xyz="0 0 0" rpy="0 0 0"/>
     <geometry>
       <mesh filename="file://$(find Robot_description)/meshes/Robot_Dog_Tibia_Another__1__1.stl" scale="0.001 0.001 0.001"/>
@@ -238,5 +238,5 @@
   </visual>
   <collision>
-    <origin xyz="0.008089 0.058658 -0.155336" rpy="0 0 0"/>
+    <origin xyz="0 0 0" rpy="0 0 0"/>
     <geometry>
       <mesh filename="file://$(find Robot_description)/meshes/Robot_Dog_Tibia_Another__1__1.stl" scale="0.001 0.001 0.001"/>
@@ -251,5 +251,5 @@
   </inertial>
   <visual>
-    <origin xyz="-0.153555 0.058358 -0.155336" rpy="0 0 0"/>
+    <origin xyz="0 0 0" rpy="0 0 0"/>
     <geometry>
       <mesh filename="file://$(find Robot_description)/meshes/Robot_Dog_Tibia_Another_1.stl" scale="0.001 0.001 0.001"/>
@@ -258,5 +258,5 @@
   </visual>
   <collision>
-    <origin xyz="-0.153555 0.058358 -0.155336" rpy="0 0 0"/>
+    <origin xyz="0 0 0" rpy="0 0 0"/>
     <geometry>
       <mesh filename="file://$(find Robot_description)/meshes/Robot_Dog_Tibia_Another_1.stl" scale="0.001 0.001 0.001"/>
@@ -271,5 +271,5 @@
   </inertial>
   <visual>
-    <origin xyz="-0.062802 -0.007845 -0.151336" rpy="0 0 0"/>
+    <origin xyz="0 0 0" rpy="0 0 0"/>
     <geometry>
       <mesh filename="file://$(find Robot_description)/meshes/Robot_Dog_Knee_Motor_to_Link_Joint__1__1.stl" scale="0.001 0.001 0.001"/>
@@ -278,5 +278,5 @@
   </visual>
   <collision>
-    <origin xyz="-0.062802 -0.007845 -0.151336" rpy="0 0 0"/>
+    <origin xyz="0 0 0" rpy="0 0 0"/>
     <geometry>
       <mesh filename="file://$(find Robot_description)/meshes/Robot_Dog_Knee_Motor_to_Link_Joint__1__1.stl" scale="0.001 0.001 0.001"/>
@@ -291,5 +291,5 @@
   </inertial>
   <visual>
-    <origin xyz="-0.062442 -0.007445 0.153336" rpy="0 0 0"/>
+    <origin xyz="0 0 0" rpy="0 0 0"/>
     <geometry>
       <mesh filename="file://$(find Robot_description)/meshes/Robot_Dog_Knee_Motor_to_Link_Joint__2__1.stl" scale="0.001 0.001 0.001"/>
@@ -298,5 +298,5 @@
   </visual>
   <collision>
-    <origin xyz="-0.062442 -0.007445 0.153336" rpy="0 0 0"/>
+    <origin xyz="0 0 0" rpy="0 0 0"/>
     <geometry>
       <mesh filename="file://$(find Robot_description)/meshes/Robot_Dog_Knee_Motor_to_Link_Joint__2__1.stl" scale="0.001 0.001 0.001"/>
