Commit message: Update Robot.xacro with relative visual origins

File: Robot_description/urdf/Robot.xacro (robot description, xacro)
@@ -31,5 +31,5 @@
   </inertial>
   <visual>
-    <origin xyz="-0.080400 0.022850 0.075328" rpy="-3.141593 1.570796 0.000000"/>
+    <origin xyz="0 0 0" rpy="-3.141593 1.570796 0.000000"/>
     <geometry>
       <mesh filename="file://$(find Robot_description)/meshes/Dynamixel_AX12a_1.stl" scale="0.001 0.001 0.001"/>
@@ -38,5 +38,5 @@
   </visual>
   <collision>
-    <origin xyz="-0.080400 0.022850 0.075328" rpy="-3.141593 1.570796 0.000000"/>
+    <origin xyz="0 0 0" rpy="-3.141593 1.570796 0.000000"/>
     <geometry>
       <mesh filename="file://$(find Robot_description)/meshes/Dynamixel_AX12a_1.stl" scale="0.001 0.001 0.001"/>
@@ -51,5 +51,5 @@
   </inertial>
   <visual>
-    <origin xyz="-0.081200 0.022850 -0.075328" rpy="0.000000 -1.570796 0.000000"/>
+    <origin xyz="0 0 0" rpy="0.000000 -1.570796 0.000000"/>
     <geometry>
       <mesh filename="file://$(find Robot_description)/meshes/Dynamixel_AX12a__1__1.stl" scale="0.001 0.001 0.001"/>
@@ -58,5 +58,5 @@
   </visual>
   <collision>
-    <origin xyz="-0.081200 0.022850 -0.075328" rpy="0.000000 -1.570796 0.000000"/>
+    <origin xyz="0 0 0" rpy="0.000000 -1.570796 0.000000"/>
     <geometry>
       <mesh filename="file://$(find Robot_description)/meshes/Dynamixel_AX12a__1__1.stl" scale="0.001 0.001 0.001"/>
@@ -71,5 +71,5 @@
   </inertial>
   <visual>
-    <origin xyz="0.081200 0.022850 0.075328" rpy="0.000000 1.570796 0.000000"/>
+    <origin xyz="0 0 0" rpy="0.000000 1.570796 0.000000"/>
     <geometry>
       <mesh filename="file://$(find Robot_description)/meshes/Dynamixel_AX12a__2__1.stl" scale="0.001 0.001 0.001"/>
@@ -78,5 +78,5 @@
   </visual>
   <collision>
-    <origin xyz="0.081200 0.022850 0.075328" rpy="0.000000 1.570796 0.000000"/>
+    <origin xyz="0 0 0" rpy="0.000000 1.570796 0.000000"/>
     <geometry>
       <mesh filename="file://$(find Robot_description)/meshes/Dynamixel_AX12a__2__1.stl" scale="0.001 0.001 0.001"/>
@@ -91,5 +91,5 @@
   </inertial>
   <visual>
-    <origin xyz="0.081200 0.022850 -0.075328" rpy="3.141593 -1.570796 0.000000"/>
+    <origin xyz="0 0 0" rpy="3.141593 -1.570796 0.000000"/>
     <geometry>
       <mesh filename="file://$(find Robot_description)/meshes/Dynamixel_AX12a__3__1.stl" scale="0.001 0.001 0.001"/>
@@ -98,5 +98,5 @@
   </visual>
   <collision>
-    <origin xyz="0.081200 0.022850 -0.075328" rpy="3.141593 -1.570796 0.000000"/>
+    <origin xyz="0 0 0" rpy="3.141593 -1.570796 0.000000"/>
     <geometry>
       <mesh filename="file://$(find Robot_description)/meshes/Dynamixel_AX12a__3__1.stl" scale="0.001 0.001 0.001"/>
@@ -111,5 +111,5 @@
   </inertial>
   <visual>
-    <origin xyz="-0.023294 -0.046310 0.173336" rpy="-1.570796 0.000000 2.094395"/>
+    <origin xyz="0 0 0" rpy="-1.570796 0.000000 2.094395"/>
     <geometry>
       <mesh filename="file://$(find Robot_description)/meshes/Robot_Dog_femur__3__1.stl" scale="0.001 0.001 0.001"/>
@@ -118,5 +118,5 @@
   </visual>
   <collision>
-    <origin xyz="-0.023294 -0.046310 0.173336" rpy="-1.570796 0.000000 2.094395"/>
+    <origin xyz="0 0 0" rpy="-1.570796 0.000000 2.094395"/>
     <geometry>
       <mesh filename="file://$(find Robot_description)/meshes/Robot_Dog_femur__3__1.stl" scale="0.001 0.001 0.001"/>
@@ -131,5 +131,5 @@
   </inertial>
   <visual>
-    <origin xyz="0.138350 -0.046010 0.173336" rpy="-1.570796 0.000000 2.094395"/>
+    <origin xyz="0 0 0" rpy="-1.570796 0.000000 2.094395"/>
     <geometry>
       <mesh filename="file://$(find Robot_description)/meshes/Robot_Dog_femur_1.stl" scale="0.001 0.001 0.001"/>
@@ -138,5 +138,5 @@
   </visual>
   <collision>
-    <origin xyz="0.138350 -0.046010 0.173336" rpy="-1.570796 0.000000 2.094395"/>
+    <origin xyz="0 0 0" rpy="-1.570796 0.000000 2.094395"/>
     <geometry>
       <mesh filename="file://$(find Robot_description)/meshes/Robot_Dog_femur_1.stl" scale="0.001 0.001 0.001"/>
@@ -151,5 +151,5 @@
   </inertial>
   <visual>
-    <origin xyz="-0.011043 -0.039232 -0.173336" rpy="1.570796 0.000000 2.094395"/>
+    <origin xyz="0 0 0" rpy="1.570796 0.000000 2.094395"/>
     <geometry>
       <mesh filename="file://$(find Robot_description)/meshes/Robot_Dog_femur__2__1.stl" scale="0.001 0.001 0.001"/>
@@ -158,5 +158,5 @@
   </visual>
   <collision>
-    <origin xyz="-0.011043 -0.039232 -0.173336" rpy="1.570796 0.000000 2.094395"/>
+    <origin xyz="0 0 0" rpy="1.570796 0.000000 2.094395"/>
     <geometry>
       <mesh filename="file://$(find Robot_description)/meshes/Robot_Dog_femur__2__1.stl" scale="0.001 0.001 0.001"/>
@@ -171,5 +171,5 @@
   </inertial>
   <visual>
-    <origin xyz="0.150249 -0.039332 -0.173336" rpy="1.570796 0.000000 2.094395"/>
+    <origin xyz="0 0 0" rpy="1.570796 0.000000 2.094395"/>
     <geometry>
       <mesh filename="file://$(find Robot_description)/meshes/Robot_Dog_femur__1__1.stl" scale="0.001 0.001 0.001"/>
@@ -178,5 +178,5 @@
   </visual>
   <collision>
-    <origin xyz="0.150249 -0.039332 -0.173336" rpy="1.570796 0.000000 2.094395"/>
+    <origin xyz="0 0 0" rpy="1.570796 0.000000 2.094395"/>
     <geometry>
       <mesh filename="file://$(find Robot_description)/meshes/Robot_Dog_femur__1__1.stl" scale="0.001 0.001 0.001"/>
@@ -191,5 +191,5 @@
   </inertial>
   <visual>
-    <origin xyz="-0.026786 -0.085078 -0.155336" rpy="-1.570796 0.000000 1.047198"/>
+    <origin xyz="0 0 0" rpy="-1.570796 0.000000 1.047198"/>
     <geometry>
       <mesh filename="file://$(find Robot_description)/meshes/Robot_Dog_TIBIA_1.stl" scale="0.001 0.001 0.001"/>
@@ -198,5 +198,5 @@
   </visual>
   <collision>
-    <origin xyz="-0.026786 -0.085078 -0.155336" rpy="-1.570796 0.000000 1.047198"/>
+    <origin xyz="0 0 0" rpy="-1.570796 0.000000 1.047198"/>
     <geometry>
       <mesh filename="file://$(find Robot_description)/meshes/Robot_Dog_TIBIA_1.stl" scale="0.001 0.001 0.001"/>
@@ -211,5 +211,5 @@
   </inertial>
   <visual>
-    <origin xyz="0.134506 -0.085178 -0.155336" rpy="-1.570796 0.000000 1.047198"/>
+    <origin xyz="0 0 0" rpy="-1.570796 0.000000 1.047198"/>
     <geometry>
       <mesh filename="file://$(find Robot_description)/meshes/Robot_Dog_TIBIA__1__1.stl" scale="0.001 0.001 0.001"/>
@@ -218,5 +218,5 @@
   </visual>
   <collision>
-    <origin xyz="0.134506 -0.085178 -0.155336" rpy="-1.570796 0.000000 1.047198"/>
+    <origin xyz="0 0 0" rpy="-1.570796 0.000000 1.047198"/>
     <geometry>
       <mesh filename="file://$(find Robot_description)/meshes/Robot_Dog_TIBIA__1__1.stl" scale="0.001 0.001 0.001"/>
@@ -231,5 +231,5 @@
   </inertial>
   <visual>
-    <origin xyz="-0.026924 -0.085162 0.170836" rpy="-1.570796 0.000000 1.047198"/>
+    <origin xyz="0 0 0" rpy="-1.570796 0.000000 1.047198"/>
     <geometry>
       <mesh filename="file://$(find Robot_description)/meshes/Robot_Dog_Tibia_Another__1__1.stl" scale="0.001 0.001 0.001"/>
@@ -238,5 +238,5 @@
   </visual>
   <collision>
-    <origin xyz="-0.026924 -0.085162 0.170836" rpy="-1.570796 0.000000 1.047198"/>
+    <origin xyz="0 0 0" rpy="-1.570796 0.000000 1.047198"/>
     <geometry>
       <mesh filename="file://$(find Robot_description)/meshes/Robot_Dog_Tibia_Another__1__1.stl" scale="0.001 0.001 0.001"/>
@@ -251,5 +251,5 @@
   </inertial>
   <visual>
-    <origin xyz="0.134720 -0.084862 0.170836" rpy="-1.570796 0.000000 1.047198"/>
+    <origin xyz="0 0 0" rpy="-1.570796 0.000000 1.047198"/>
     <geometry>
       <mesh filename="file://$(find Robot_description)/meshes/Robot_Dog_Tibia_Another_1.stl" scale="0.001 0.001 0.001"/>
@@ -258,5 +258,5 @@
   </visual>
   <collision>
-    <origin xyz="0.134720 -0.084862 0.170836" rpy="-1.570796 0.000000 1.047198"/>
+    <origin xyz="0 0 0" rpy="-1.570796 0.000000 1.047198"/>
     <geometry>
       <mesh filename="file://$(find Robot_description)/meshes/Robot_Dog_Tibia_Another_1.stl" scale="0.001 0.001 0.001"/>
@@ -271,5 +271,5 @@
   </inertial>
   <visual>
-    <origin xyz="0.028428 -0.033149 0.152836" rpy="1.570796 0.000000 0.872665"/>
+    <origin xyz="0 0 0" rpy="1.570796 0.000000 0.872665"/>
     <geometry>
       <mesh filename="file://$(find Robot_description)/meshes/Robot_Dog_Knee_Motor_to_Link_Joint__1__1.stl" scale="0.001 0.001 0.001"/>
@@ -278,5 +278,5 @@
   </visual>
   <collision>
-    <origin xyz="0.028428 -0.033149 0.152836" rpy="1.570796 0.000000 0.872665"/>
+    <origin xyz="0 0 0" rpy="1.570796 0.000000 0.872665"/>
     <geometry>
       <mesh filename="file://$(find Robot_description)/meshes/Robot_Dog_Knee_Motor_to_Link_Joint__1__1.stl" scale="0.001 0.001 0.001"/>
@@ -291,5 +291,5 @@
   </inertial>
   <visual>
-    <origin xyz="0.028040 -0.033525 -0.154836" rpy="-1.570796 0.000000 0.872665"/>
+    <origin xyz="0 0 0" rpy="-1.570796 0.000000 0.872665"/>
     <geometry>
       <mesh filename="file://$(find Robot_description)/meshes/Robot_Dog_Knee_Motor_to_Link_Joint__2__1.stl" scale="0.001 0.001 0.001"/>
@@ -298,5 +298,5 @@
   </visual>
   <collision>
-    <origin xyz="0.028040 -0.033525 -0.154836" rpy="-1.570796 0.000000 0.872665"/>
+    <origin xyz="0 0 0" rpy="-1.570796 0.000000 0.872665"/>
     <geometry>
       <mesh filename="file://$(find Robot_description)/meshes/Robot_Dog_Knee_Motor_to_Link_Joint__2__1.stl" scale="0.001 0.001 0.001"/>
@@ -311,5 +311,5 @@
   </inertial>
   <visual>
-    <origin xyz="-0.133252 -0.033425 -0.154836" rpy="-1.570796 0.000000 0.872665"/>
+    <origin xyz="0 0 0" rpy="-1.570796 0.000000 0.872665"/>
     <geometry>
       <mesh filename="file://$(find Robot_description)/meshes/Robot_Dog_Knee_Motor_to_Link_Joint__3__1.stl" scale="0.001 0.001 0.001"/>
@@ -318,5 +318,5 @@
   </visual>
   <collision>
-    <origin xyz="-0.133252 -0.033425 -0.154836" rpy="-1.570796 0.000000 0.872665"/>
+    <origin xyz="0 0 0" rpy="-1.570796 0.000000 0.872665"/>
     <geometry>
       <mesh filename="file://$(find Robot_description)/meshes/Robot_Dog_Knee_Motor_to_Link_Joint__3__1.stl" scale="0.001 0.001 0.001"/>
@@ -331,5 +331,5 @@
   </inertial>
   <visual>
-    <origin xyz="-0.133216 -0.033449 0.154836" rpy="1.570796 0.000000 0.872665"/>
+    <origin xyz="0 0 0" rpy="1.570796 0.000000 0.872665"/>
     <geometry>
       <mesh filename="file://$(find Robot_description)/meshes/Robot_Dog_Knee_Motor_to_Link_Joint_1.stl" scale="0.001 0.001 0.001"/>
@@ -338,5 +338,5 @@
   </visual>
   <collision>
-    <origin xyz="-0.133216 -0.033449 0.154836" rpy="1.570796 0.000000 0.872665"/>
+    <origin xyz="0 0 0" rpy="1.570796 0.000000 0.872665"/>
     <geometry>
       <mesh filename="file://$(find Robot_description)/meshes/Robot_Dog_Knee_Motor_to_Link_Joint_1.stl" scale="0.001 0.001 0.001"/>
@@ -351,5 +351,5 @@
   </inertial>
   <visual>
-    <origin xyz="-0.071587 -0.049411 0.160336" rpy="1.570796 0.000000 -0.760964"/>
+    <origin xyz="0 0 0" rpy="1.570796 0.000000 -0.760964"/>
     <geometry>
       <mesh filename="file://$(find Robot_description)/meshes/Robot_Dog_Tibia_Hip_Link_1.stl" scale="0.001 0.001 0.001"/>
@@ -358,5 +358,5 @@
   </visual>
   <collision>
-    <origin xyz="-0.071587 -0.049411 0.160336" rpy="1.570796 0.000000 -0.760964"/>
+    <origin xyz="0 0 0" rpy="1.570796 0.000000 -0.760964"/>
     <geometry>
       <mesh filename="file://$(find Robot_description)/meshes/Robot_Dog_Tibia_Hip_Link_1.stl" scale="0.001 0.001 0.001"/>
@@ -371,5 +371,5 @@
   </inertial>
   <visual>
-    <origin xyz="0.090057 -0.049111 0.158336" rpy="1.570796 0.000000 -0.760964"/>
+    <origin xyz="0 0 0" rpy="1.570796 0.000000 -0.760964"/>
     <geometry>
       <mesh filename="file://$(find Robot_description)/meshes/Robot_Dog_Tibia_Hip_Link__1__1.stl" scale="0.001 0.001 0.001"/>
@@ -378,5 +378,5 @@
   </visual>
   <collision>
-    <origin xyz="0.090057 -0.049111 0.158336" rpy="1.570796 0.000000 -0.760964"/>
+    <origin xyz="0 0 0" rpy="1.570796 0.000000 -0.760964"/>
     <geometry>
       <mesh filename="file://$(find Robot_description)/meshes/Robot_Dog_Tibia_Hip_Link__1__1.stl" scale="0.001 0.001 0.001"/>
@@ -391,5 +391,5 @@
   </inertial>
   <visual>
-    <origin xyz="-0.075043 -0.053032 -0.160336" rpy="-1.570796 0.000000 -0.760964"/>
+    <origin xyz="0 0 0" rpy="-1.570796 0.000000 -0.760964"/>
     <geometry>
       <mesh filename="file://$(find Robot_description)/meshes/Robot_Dog_Tibia_Hip_Link__2__1.stl" scale="0.001 0.001 0.001"/>
@@ -398,5 +398,5 @@
   </visual>
   <collision>
-    <origin xyz="-0.075043 -0.053032 -0.160336" rpy="-1.570796 0.000000 -0.760964"/>
+    <origin xyz="0 0 0" rpy="-1.570796 0.000000 -0.760964"/>
     <geometry>
       <mesh filename="file://$(find Robot_description)/meshes/Robot_Dog_Tibia_Hip_Link__2__1.stl" scale="0.001 0.001 0.001"/>
@@ -411,5 +411,5 @@
   </inertial>
   <visual>
-    <origin xyz="0.086249 -0.053132 -0.160336" rpy="-1.570796 0.000000 -0.760964"/>
+    <origin xyz="0 0 0" rpy="-1.570796 0.000000 -0.760964"/>
     <geometry>
       <mesh filename="file://$(find Robot_description)/meshes/Robot_Dog_Tibia_Hip_Link__3__1.stl" scale="0.001 0.001 0.001"/>
@@ -418,5 +418,5 @@
   </visual>
   <collision>
-    <origin xyz="0.086249 -0.053132 -0.160336" rpy="-1.570796 0.000000 -0.760964"/>
+    <origin xyz="0 0 0" rpy="-1.570796 0.000000 -0.760964"/>
     <geometry>
       <mesh filename="file://$(find Robot_description)/meshes/Robot_Dog_Tibia_Hip_Link__3__1.stl" scale="0.001 0.001 0.001"/>
@@ -431,5 +431,5 @@
   </inertial>
   <visual>
-    <origin xyz="-0.067532 -0.162176 0.163086" rpy="0.000000 0.000000 -0.523599"/>
+    <origin xyz="0 0 0" rpy="0.000000 0.000000 -0.523599"/>
     <geometry>
       <mesh filename="file://$(find Robot_description)/meshes/Foot2_1.stl" scale="0.001 0.001 0.001"/>
@@ -438,5 +438,5 @@
   </visual>
   <collision>
-    <origin xyz="-0.067532 -0.162176 0.163086" rpy="0.000000 0.000000 -0.523599"/>
+    <origin xyz="0 0 0" rpy="0.000000 0.000000 -0.523599"/>
     <geometry>
       <mesh filename="file://$(find Robot_description)/meshes/Foot2_1.stl" scale="0.001 0.001 0.001"/>
@@ -451,5 +451,5 @@
   </inertial>
   <visual>
-    <origin xyz="0.094112 -0.161876 0.163086" rpy="0.000000 0.000000 -0.523599"/>
+    <origin xyz="0 0 0" rpy="0.000000 0.000000 -0.523599"/>
     <geometry>
       <mesh filename="file://$(find Robot_description)/meshes/Foot2__1__1.stl" scale="0.001 0.001 0.001"/>
@@ -458,5 +458,5 @@
   </visual>
   <collision>
-    <origin xyz="0.094112 -0.161876 0.163086" rpy="0.000000 0.000000 -0.523599"/>
+    <origin xyz="0 0 0" rpy="0.000000 0.000000 -0.523599"/>
     <geometry>
       <mesh filename="file://$(find Robot_description)/meshes/Foot2__1__1.stl" scale="0.001 0.001 0.001"/>
@@ -471,5 +471,5 @@
   </inertial>
   <visual>
-    <origin xyz="-0.067394 -0.162092 -0.163086" rpy="0.000000 0.000000 -0.523599"/>
+    <origin xyz="0 0 0" rpy="0.000000 0.000000 -0.523599"/>
     <geometry>
       <mesh filename="file://$(find Robot_description)/meshes/Foot2__2__1.stl" scale="0.001 0.001 0.001"/>
@@ -478,5 +478,5 @@
   </visual>
   <collision>
-    <origin xyz="-0.067394 -0.162092 -0.163086" rpy="0.000000 0.000000 -0.523599"/>
+    <origin xyz="0 0 0" rpy="0.000000 0.000000 -0.523599"/>
     <geometry>
       <mesh filename="file://$(find Robot_description)/meshes/Foot2__2__1.stl" scale="0.001 0.001 0.001"/>
@@ -491,5 +491,5 @@
   </inertial>
   <visual>
-    <origin xyz="0.093898 -0.162192 -0.163086" rpy="0.000000 0.000000 -0.523599"/>
+    <origin xyz="0 0 0" rpy="0.000000 0.000000 -0.523599"/>
     <geometry>
       <mesh filename="file://$(find Robot_description)/meshes/Foot2__3__1.stl" scale="0.001 0.001 0.001"/>
@@ -498,5 +498,5 @@
   </visual>
   <collision>
-    <origin xyz="0.093898 -0.162192 -0.163086" rpy="0.000000 0.000000 -0.523599"/>
+    <origin xyz="0 0 0" rpy="0.000000 0.000000 -0.523599"/>
     <geometry>
       <mesh filename="file://$(find Robot_description)/meshes/Foot2__3__1.stl" scale="0.001 0.001 0.001"/>
@@ -511,5 +511,5 @@
   </inertial>
   <visual>
-    <origin xyz="0.000000 -0.005000 -0.000000" rpy="0 0 0"/>
+    <origin xyz="0 0 0" rpy="0.000000 0.000000 0.000000"/>
     <geometry>
       <mesh filename="file://$(find Robot_description)/meshes/Battery_Equivalent_1.stl" scale="0.001 0.001 0.001"/>
@@ -518,5 +518,5 @@
   </visual>
   <collision>
-    <origin xyz="0.000000 -0.005000 -0.000000" rpy="0 0 0"/>
+    <origin xyz="0 0 0" rpy="0.000000 0.000000 0.000000"/>
     <geometry>
       <mesh filename="file://$(find Robot_description)/meshes/Battery_Equivalent_1.stl" scale="0.001 0.001 0.001"/>
@@ -531,5 +531,5 @@
   </inertial>
   <visual>
-    <origin xyz="0.099902 0.037245 0.132236" rpy="0.000000 0.000000 -1.570796"/>
+    <origin xyz="0 0 0" rpy="0.000000 0.000000 -1.570796"/>
     <geometry>
       <mesh filename="file://$(find Robot_description)/meshes/Dynamixel_AX12a__1___7__1.stl" scale="0.001 0.001 0.001"/>
@@ -538,5 +538,5 @@
   </visual>
   <collision>
-    <origin xyz="0.099902 0.037245 0.132236" rpy="0.000000 0.000000 -1.570796"/>
+    <origin xyz="0 0 0" rpy="0.000000 0.000000 -1.570796"/>
     <geometry>
       <mesh filename="file://$(find Robot_description)/meshes/Dynamixel_AX12a__1___7__1.stl" scale="0.001 0.001 0.001"/>
@@ -551,5 +551,5 @@
   </inertial>
   <visual>
-    <origin xyz="0.061702 0.007245 0.132236" rpy="0.000000 0.000000 1.570796"/>
+    <origin xyz="0 0 0" rpy="0.000000 0.000000 1.570796"/>
     <geometry>
       <mesh filename="file://$(find Robot_description)/meshes/Dynamixel_AX12a__1___8__1.stl" scale="0.001 0.001 0.001"/>
@@ -558,5 +558,5 @@
   </visual>
   <collision>
-    <origin xyz="0.061702 0.007245 0.132236" rpy="0.000000 0.000000 1.570796"/>
+    <origin xyz="0 0 0" rpy="0.000000 0.000000 1.570796"/>
     <geometry>
       <mesh filename="file://$(find Robot_description)/meshes/Dynamixel_AX12a__1___8__1.stl" scale="0.001 0.001 0.001"/>
@@ -571,5 +571,5 @@
   </inertial>
   <visual>
-    <origin xyz="-0.061742 0.036945 0.132236" rpy="0.000000 0.000000 -1.570796"/>
+    <origin xyz="0 0 0" rpy="0.000000 0.000000 -1.570796"/>
     <geometry>
       <mesh filename="file://$(find Robot_description)/meshes/Dynamixel_AX12a__1___3__1.stl" scale="0.001 0.001 0.001"/>
@@ -578,5 +578,5 @@
   </visual>
   <collision>
-    <origin xyz="-0.061742 0.036945 0.132236" rpy="0.000000 0.000000 -1.570796"/>
+    <origin xyz="0 0 0" rpy="0.000000 0.000000 -1.570796"/>
     <geometry>
       <mesh filename="file://$(find Robot_description)/meshes/Dynamixel_AX12a__1___3__1.stl" scale="0.001 0.001 0.001"/>
@@ -591,5 +591,5 @@
   </inertial>
   <visual>
-    <origin xyz="-0.099942 0.006945 0.132236" rpy="0.000000 0.000000 1.570796"/>
+    <origin xyz="0 0 0" rpy="0.000000 0.000000 1.570796"/>
     <geometry>
       <mesh filename="file://$(find Robot_description)/meshes/Dynamixel_AX12a__1___4__1.stl" scale="0.001 0.001 0.001"/>
@@ -598,5 +598,5 @@
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