Commit message: Manually tune motor boxes visual and collision origins

File: Robot_description/urdf/Robot.xacro (robot description, xacro)
@@ -31,5 +31,5 @@
   </inertial>
   <visual>
-    <origin xyz="0 0 0" rpy="0 0 0"/>
+    <origin xyz="-0.016000 0.015000 0.034000" rpy="-3.141593 1.570796 0.000000"/>
     <geometry>
       <mesh filename="file://$(find Robot_description)/meshes/Dynamixel_AX12a_1.stl" scale="0.001 0.001 0.001"/>
@@ -38,5 +38,5 @@
   </visual>
   <collision>
-    <origin xyz="0 0 0" rpy="0 0 0"/>
+    <origin xyz="-0.016000 0.015000 0.034000" rpy="-3.141593 1.570796 0.000000"/>
     <geometry>
       <mesh filename="file://$(find Robot_description)/meshes/Dynamixel_AX12a_1.stl" scale="0.001 0.001 0.001"/>
@@ -51,5 +51,5 @@
   </inertial>
   <visual>
-    <origin xyz="0 0 0" rpy="0 0 0"/>
+    <origin xyz="0.016000 -0.015000 -0.034000" rpy="-0.000000 -1.570796 0.000000"/>
     <geometry>
       <mesh filename="file://$(find Robot_description)/meshes/Dynamixel_AX12a__1__1.stl" scale="0.001 0.001 0.001"/>
@@ -58,5 +58,5 @@
   </visual>
   <collision>
-    <origin xyz="0 0 0" rpy="0 0 0"/>
+    <origin xyz="0.016000 -0.015000 -0.034000" rpy="-0.000000 -1.570796 0.000000"/>
     <geometry>
       <mesh filename="file://$(find Robot_description)/meshes/Dynamixel_AX12a__1__1.stl" scale="0.001 0.001 0.001"/>
@@ -71,5 +71,5 @@
   </inertial>
   <visual>
-    <origin xyz="0 0 0" rpy="0 0 0"/>
+    <origin xyz="-0.016000 0.015000 0.034000" rpy="-0.000000 1.570796 0.000000"/>
     <geometry>
       <mesh filename="file://$(find Robot_description)/meshes/Dynamixel_AX12a__2__1.stl" scale="0.001 0.001 0.001"/>
@@ -78,5 +78,5 @@
   </visual>
   <collision>
-    <origin xyz="0 0 0" rpy="0 0 0"/>
+    <origin xyz="-0.016000 0.015000 0.034000" rpy="-0.000000 1.570796 0.000000"/>
     <geometry>
       <mesh filename="file://$(find Robot_description)/meshes/Dynamixel_AX12a__2__1.stl" scale="0.001 0.001 0.001"/>
@@ -91,5 +91,5 @@
   </inertial>
   <visual>
-    <origin xyz="0 0 0" rpy="0 0 0"/>
+    <origin xyz="-0.016000 0.015000 -0.034000" rpy="3.141593 -1.570796 0.000000"/>
     <geometry>
       <mesh filename="file://$(find Robot_description)/meshes/Dynamixel_AX12a__3__1.stl" scale="0.001 0.001 0.001"/>
@@ -98,5 +98,5 @@
   </visual>
   <collision>
-    <origin xyz="0 0 0" rpy="0 0 0"/>
+    <origin xyz="-0.016000 0.015000 -0.034000" rpy="3.141593 -1.570796 0.000000"/>
     <geometry>
       <mesh filename="file://$(find Robot_description)/meshes/Dynamixel_AX12a__3__1.stl" scale="0.001 0.001 0.001"/>
@@ -111,5 +111,5 @@
   </inertial>
   <visual>
-    <origin xyz="0 0 0" rpy="0 0 0"/>
+    <origin xyz="0.039548 -0.082655 0.020000" rpy="-1.570796 0.000000 2.094395"/>
     <geometry>
       <mesh filename="file://$(find Robot_description)/meshes/Robot_Dog_femur__3__1.stl" scale="0.001 0.001 0.001"/>
@@ -118,5 +118,5 @@
   </visual>
   <collision>
-    <origin xyz="0 0 0" rpy="0 0 0"/>
+    <origin xyz="0.039548 -0.082655 0.020000" rpy="-1.570796 0.000000 2.094395"/>
     <geometry>
       <mesh filename="file://$(find Robot_description)/meshes/Robot_Dog_femur__3__1.stl" scale="0.001 0.001 0.001"/>
@@ -131,5 +131,5 @@
   </inertial>
   <visual>
-    <origin xyz="0 0 0" rpy="0 0 0"/>
+    <origin xyz="0.039548 -0.082655 0.020000" rpy="-1.570796 0.000000 2.094395"/>
     <geometry>
       <mesh filename="file://$(find Robot_description)/meshes/Robot_Dog_femur_1.stl" scale="0.001 0.001 0.001"/>
@@ -138,5 +138,5 @@
   </visual>
   <collision>
-    <origin xyz="0 0 0" rpy="0 0 0"/>
+    <origin xyz="0.039548 -0.082655 0.020000" rpy="-1.570796 0.000000 2.094395"/>
     <geometry>
       <mesh filename="file://$(find Robot_description)/meshes/Robot_Dog_femur_1.stl" scale="0.001 0.001 0.001"/>
@@ -151,5 +151,5 @@
   </inertial>
   <visual>
-    <origin xyz="0 0 0" rpy="0 0 0"/>
+    <origin xyz="0.051807 -0.075577 -0.020000" rpy="1.570796 -0.000000 2.094395"/>
     <geometry>
       <mesh filename="file://$(find Robot_description)/meshes/Robot_Dog_femur__2__1.stl" scale="0.001 0.001 0.001"/>
@@ -158,5 +158,5 @@
   </visual>
   <collision>
-    <origin xyz="0 0 0" rpy="0 0 0"/>
+    <origin xyz="0.051807 -0.075577 -0.020000" rpy="1.570796 -0.000000 2.094395"/>
     <geometry>
       <mesh filename="file://$(find Robot_description)/meshes/Robot_Dog_femur__2__1.stl" scale="0.001 0.001 0.001"/>
@@ -171,5 +171,5 @@
   </inertial>
   <visual>
-    <origin xyz="0 0 0" rpy="0 0 0"/>
+    <origin xyz="0.051807 -0.075577 -0.020000" rpy="1.570796 -0.000000 2.094395"/>
     <geometry>
       <mesh filename="file://$(find Robot_description)/meshes/Robot_Dog_femur__1__1.stl" scale="0.001 0.001 0.001"/>
@@ -178,5 +178,5 @@
   </visual>
   <collision>
-    <origin xyz="0 0 0" rpy="0 0 0"/>
+    <origin xyz="0.051807 -0.075577 -0.020000" rpy="1.570796 -0.000000 2.094395"/>
     <geometry>
       <mesh filename="file://$(find Robot_description)/meshes/Robot_Dog_femur__1__1.stl" scale="0.001 0.001 0.001"/>
@@ -191,5 +191,5 @@
   </inertial>
   <visual>
-    <origin xyz="0 0 0" rpy="0 0 0"/>
+    <origin xyz="-0.018835 -0.026504 -0.000000" rpy="-1.570796 -0.000000 1.047198"/>
     <geometry>
       <mesh filename="file://$(find Robot_description)/meshes/Robot_Dog_TIBIA_1.stl" scale="0.001 0.001 0.001"/>
@@ -198,5 +198,5 @@
   </visual>
   <collision>
-    <origin xyz="0 0 0" rpy="0 0 0"/>
+    <origin xyz="-0.018835 -0.026504 -0.000000" rpy="-1.570796 -0.000000 1.047198"/>
     <geometry>
       <mesh filename="file://$(find Robot_description)/meshes/Robot_Dog_TIBIA_1.stl" scale="0.001 0.001 0.001"/>
@@ -211,5 +211,5 @@
   </inertial>
   <visual>
-    <origin xyz="0 0 0" rpy="0 0 0"/>
+    <origin xyz="-0.018835 -0.026504 -0.000000" rpy="-1.570796 -0.000000 1.047198"/>
     <geometry>
       <mesh filename="file://$(find Robot_description)/meshes/Robot_Dog_TIBIA__1__1.stl" scale="0.001 0.001 0.001"/>
@@ -218,5 +218,5 @@
   </visual>
   <collision>
-    <origin xyz="0 0 0" rpy="0 0 0"/>
+    <origin xyz="-0.018835 -0.026504 -0.000000" rpy="-1.570796 -0.000000 1.047198"/>
     <geometry>
       <mesh filename="file://$(find Robot_description)/meshes/Robot_Dog_TIBIA__1__1.stl" scale="0.001 0.001 0.001"/>
@@ -231,5 +231,5 @@
   </inertial>
   <visual>
-    <origin xyz="0 0 0" rpy="0 0 0"/>
+    <origin xyz="-0.018835 -0.026504 0.015500" rpy="-1.570796 0.000000 1.047198"/>
     <geometry>
       <mesh filename="file://$(find Robot_description)/meshes/Robot_Dog_Tibia_Another__1__1.stl" scale="0.001 0.001 0.001"/>
@@ -238,5 +238,5 @@
   </visual>
   <collision>
-    <origin xyz="0 0 0" rpy="0 0 0"/>
+    <origin xyz="-0.018835 -0.026504 0.015500" rpy="-1.570796 0.000000 1.047198"/>
     <geometry>
       <mesh filename="file://$(find Robot_description)/meshes/Robot_Dog_Tibia_Another__1__1.stl" scale="0.001 0.001 0.001"/>
@@ -251,5 +251,5 @@
   </inertial>
   <visual>
-    <origin xyz="0 0 0" rpy="0 0 0"/>
+    <origin xyz="-0.018835 -0.026504 0.015500" rpy="-1.570796 0.000000 1.047198"/>
     <geometry>
       <mesh filename="file://$(find Robot_description)/meshes/Robot_Dog_Tibia_Another_1.stl" scale="0.001 0.001 0.001"/>
@@ -258,5 +258,5 @@
   </visual>
   <collision>
-    <origin xyz="0 0 0" rpy="0 0 0"/>
+    <origin xyz="-0.018835 -0.026504 0.015500" rpy="-1.570796 0.000000 1.047198"/>
     <geometry>
       <mesh filename="file://$(find Robot_description)/meshes/Robot_Dog_Tibia_Another_1.stl" scale="0.001 0.001 0.001"/>
@@ -271,5 +271,5 @@
   </inertial>
   <visual>
-    <origin xyz="0 0 0" rpy="0 0 0"/>
+    <origin xyz="-0.034374 -0.040994 0.001500" rpy="1.570796 0.000000 0.872665"/>
     <geometry>
       <mesh filename="file://$(find Robot_description)/meshes/Robot_Dog_Knee_Motor_to_Link_Joint__1__1.stl" scale="0.001 0.001 0.001"/>
@@ -278,5 +278,5 @@
   </visual>
   <collision>
-    <origin xyz="0 0 0" rpy="0 0 0"/>
+    <origin xyz="-0.034374 -0.040994 0.001500" rpy="1.570796 0.000000 0.872665"/>
     <geometry>
       <mesh filename="file://$(find Robot_description)/meshes/Robot_Dog_Knee_Motor_to_Link_Joint__1__1.stl" scale="0.001 0.001 0.001"/>
@@ -291,5 +291,5 @@
   </inertial>
   <visual>
-    <origin xyz="0 0 0" rpy="0 0 0"/>
+    <origin xyz="-0.034402 -0.040970 -0.001500" rpy="-1.570796 -0.000000 0.872665"/>
     <geometry>
       <mesh filename="file://$(find Robot_description)/meshes/Robot_Dog_Knee_Motor_to_Link_Joint__2__1.stl" scale="0.001 0.001 0.001"/>
@@ -298,5 +298,5 @@
   </visual>
   <collision>
-    <origin xyz="0 0 0" rpy="0 0 0"/>
+    <origin xyz="-0.034402 -0.040970 -0.001500" rpy="-1.570796 -0.000000 0.872665"/>
     <geometry>
       <mesh filename="file://$(find Robot_description)/meshes/Robot_Dog_Knee_Motor_to_Link_Joint__2__1.stl" scale="0.001 0.001 0.001"/>
@@ -311,5 +311,5 @@
   </inertial>
   <visual>
-    <origin xyz="0.09885 -0.007545 0.153336" rpy="0 0 0"/>
+    <origin xyz="-0.034402 -0.040970 -0.001500" rpy="-1.570796 -0.000000 0.872665"/>
     <geometry>
       <mesh filename="file://$(find Robot_description)/meshes/Robot_Dog_Knee_Motor_to_Link_Joint__3__1.stl" scale="0.001 0.001 0.001"/>
@@ -318,5 +318,5 @@
   </visual>
   <collision>
-    <origin xyz="0.09885 -0.007545 0.153336" rpy="0 0 0"/>
+    <origin xyz="-0.034402 -0.040970 -0.001500" rpy="-1.570796 -0.000000 0.872665"/>
     <geometry>
       <mesh filename="file://$(find Robot_description)/meshes/Robot_Dog_Knee_Motor_to_Link_Joint__3__1.stl" scale="0.001 0.001 0.001"/>
@@ -331,5 +331,5 @@
   </inertial>
   <visual>
-    <origin xyz="0.098842 -0.007545 -0.153336" rpy="0 0 0"/>
+    <origin xyz="-0.034374 -0.040994 0.001500" rpy="1.570796 0.000000 0.872665"/>
     <geometry>
       <mesh filename="file://$(find Robot_description)/meshes/Robot_Dog_Knee_Motor_to_Link_Joint_1.stl" scale="0.001 0.001 0.001"/>
@@ -338,5 +338,5 @@
   </visual>
   <collision>
-    <origin xyz="0.098842 -0.007545 -0.153336" rpy="0 0 0"/>
+    <origin xyz="-0.034374 -0.040994 0.001500" rpy="1.570796 0.000000 0.872665"/>
     <geometry>
       <mesh filename="file://$(find Robot_description)/meshes/Robot_Dog_Knee_Motor_to_Link_Joint_1.stl" scale="0.001 0.001 0.001"/>
@@ -351,5 +351,5 @@
   </inertial>
   <visual>
-    <origin xyz="0.114912 0.011606 -0.160336" rpy="0 0 0"/>
+    <origin xyz="0.043324 -0.037805 0.000000" rpy="1.570796 -0.000000 -0.760964"/>
     <geometry>
       <mesh filename="file://$(find Robot_description)/meshes/Robot_Dog_Tibia_Hip_Link_1.stl" scale="0.001 0.001 0.001"/>
@@ -358,5 +358,5 @@
   </visual>
   <collision>
-    <origin xyz="0.114912 0.011606 -0.160336" rpy="0 0 0"/>
+    <origin xyz="0.043324 -0.037805 0.000000" rpy="1.570796 -0.000000 -0.760964"/>
     <geometry>
       <mesh filename="file://$(find Robot_description)/meshes/Robot_Dog_Tibia_Hip_Link_1.stl" scale="0.001 0.001 0.001"/>
@@ -371,5 +371,5 @@
   </inertial>
   <visual>
-    <origin xyz="-0.046732 0.011306 -0.158336" rpy="0 0 0"/>
+    <origin xyz="0.043324 -0.037805 0.000000" rpy="1.570796 -0.000000 -0.760964"/>
     <geometry>
       <mesh filename="file://$(find Robot_description)/meshes/Robot_Dog_Tibia_Hip_Link__1__1.stl" scale="0.001 0.001 0.001"/>
@@ -378,5 +378,5 @@
   </visual>
   <collision>
-    <origin xyz="-0.046732 0.011306 -0.158336" rpy="0 0 0"/>
+    <origin xyz="0.043324 -0.037805 0.000000" rpy="1.570796 -0.000000 -0.760964"/>
     <geometry>
       <mesh filename="file://$(find Robot_description)/meshes/Robot_Dog_Tibia_Hip_Link__1__1.stl" scale="0.001 0.001 0.001"/>
@@ -391,5 +391,5 @@
   </inertial>
   <visual>
-    <origin xyz="0.11492 0.011606 0.160336" rpy="0 0 0"/>
+    <origin xyz="0.039876 -0.041426 0.000000" rpy="-1.570796 0.000000 -0.760964"/>
     <geometry>
       <mesh filename="file://$(find Robot_description)/meshes/Robot_Dog_Tibia_Hip_Link__2__1.stl" scale="0.001 0.001 0.001"/>
@@ -398,5 +398,5 @@
   </visual>
   <collision>
-    <origin xyz="0.11492 0.011606 0.160336" rpy="0 0 0"/>
+    <origin xyz="0.039876 -0.041426 0.000000" rpy="-1.570796 0.000000 -0.760964"/>
     <geometry>
       <mesh filename="file://$(find Robot_description)/meshes/Robot_Dog_Tibia_Hip_Link__2__1.stl" scale="0.001 0.001 0.001"/>
@@ -411,5 +411,5 @@
   </inertial>
   <visual>
-    <origin xyz="-0.046372 0.011706 0.160336" rpy="0 0 0"/>
+    <origin xyz="0.039876 -0.041426 0.000000" rpy="-1.570796 0.000000 -0.760964"/>
     <geometry>
       <mesh filename="file://$(find Robot_description)/meshes/Robot_Dog_Tibia_Hip_Link__3__1.stl" scale="0.001 0.001 0.001"/>
@@ -418,5 +418,5 @@
   </visual>
   <collision>
-    <origin xyz="-0.046372 0.011706 0.160336" rpy="0 0 0"/>
+    <origin xyz="0.039876 -0.041426 0.000000" rpy="-1.570796 0.000000 -0.760964"/>
     <geometry>
       <mesh filename="file://$(find Robot_description)/meshes/Robot_Dog_Tibia_Hip_Link__3__1.stl" scale="0.001 0.001 0.001"/>
@@ -431,5 +431,5 @@
   </inertial>
   <visual>
-    <origin xyz="0.066532 0.160444 -0.163086" rpy="0 0 0"/>
+    <origin xyz="-0.001000 -0.001732 0.000000" rpy="-0.000000 0.000000 -0.523599"/>
     <geometry>
       <mesh filename="file://$(find Robot_description)/meshes/Foot2_1.stl" scale="0.001 0.001 0.001"/>
@@ -438,5 +438,5 @@
   </visual>
   <collision>
-    <origin xyz="0.066532 0.160444 -0.163086" rpy="0 0 0"/>
+    <origin xyz="-0.001000 -0.001732 0.000000" rpy="-0.000000 0.000000 -0.523599"/>
     <geometry>
       <mesh filename="file://$(find Robot_description)/meshes/Foot2_1.stl" scale="0.001 0.001 0.001"/>
@@ -451,5 +451,5 @@
   </inertial>
   <visual>
-    <origin xyz="-0.095112 0.160144 -0.163086" rpy="0 0 0"/>
+    <origin xyz="-0.001000 -0.001732 0.000000" rpy="-0.000000 0.000000 -0.523599"/>
     <geometry>
       <mesh filename="file://$(find Robot_description)/meshes/Foot2__1__1.stl" scale="0.001 0.001 0.001"/>
@@ -458,5 +458,5 @@
   </visual>
   <collision>
-    <origin xyz="-0.095112 0.160144 -0.163086" rpy="0 0 0"/>
+    <origin xyz="-0.001000 -0.001732 0.000000" rpy="-0.000000 0.000000 -0.523599"/>
     <geometry>
       <mesh filename="file://$(find Robot_description)/meshes/Foot2__1__1.stl" scale="0.001 0.001 0.001"/>
@@ -471,5 +471,5 @@
   </inertial>
   <visual>
-    <origin xyz="0.066394 0.16036 0.163086" rpy="0 0 0"/>
+    <origin xyz="-0.001000 -0.001732 0.000000" rpy="0.000000 0.000000 -0.523599"/>
     <geometry>
       <mesh filename="file://$(find Robot_description)/meshes/Foot2__2__1.stl" scale="0.001 0.001 0.001"/>
@@ -478,5 +478,5 @@
   </visual>
   <collision>
-    <origin xyz="0.066394 0.16036 0.163086" rpy="0 0 0"/>
+    <origin xyz="-0.001000 -0.001732 0.000000" rpy="0.000000 0.000000 -0.523599"/>
     <geometry>
       <mesh filename="file://$(find Robot_description)/meshes/Foot2__2__1.stl" scale="0.001 0.001 0.001"/>
@@ -491,5 +491,5 @@
   </inertial>
   <visual>
-    <origin xyz="-0.094898 0.16046 0.163086" rpy="0 0 0"/>
+    <origin xyz="-0.001000 -0.001732 0.000000" rpy="0.000000 0.000000 -0.523599"/>
     <geometry>
       <mesh filename="file://$(find Robot_description)/meshes/Foot2__3__1.stl" scale="0.001 0.001 0.001"/>
@@ -498,5 +498,5 @@
   </visual>
   <collision>
-    <origin xyz="-0.094898 0.16046 0.163086" rpy="0 0 0"/>
+    <origin xyz="-0.001000 -0.001732 0.000000" rpy="0.000000 0.000000 -0.523599"/>
     <geometry>
       <mesh filename="file://$(find Robot_description)/meshes/Foot2__3__1.stl" scale="0.001 0.001 0.001"/>
@@ -511,5 +511,5 @@
   </inertial>
   <visual>
-    <origin xyz="0.0 -0.005 -0.0" rpy="0 0 0"/>
+    <origin xyz="0.000000 0.000000 -0.000000" rpy="0.000000 -0.000000 0.000000"/>
     <geometry>
       <mesh filename="file://$(find Robot_description)/meshes/Battery_Equivalent_1.stl" scale="0.001 0.001 0.001"/>
@@ -518,5 +518,5 @@
   </visual>
   <collision>
-    <origin xyz="0.0 -0.005 -0.0" rpy="0 0 0"/>
+    <origin xyz="0.000000 0.000000 -0.000000" rpy="0.000000 -0.000000 0.000000"/>
     <geometry>
       <mesh filename="file://$(find Robot_description)/meshes/Battery_Equivalent_1.stl" scale="0.001 0.001 0.001"/>
@@ -531,5 +531,5 @@
   </inertial>
   <visual>
-    <origin xyz="-0.114902 -0.003245 -0.148236" rpy="0 0 0"/>
+    <origin xyz="-0.015000 0.034000 -0.016000" rpy="-0.000000 -0.000000 -1.570796"/>
     <geometry>
       <mesh filename="file://$(find Robot_description)/meshes/Dynamixel_AX12a__1___7__1.stl" scale="0.001 0.001 0.001"/>
@@ -538,5 +538,5 @@
   </visual>
   <collision>
-    <origin xyz="-0.114902 -0.003245 -0.148236" rpy="0 0 0"/>
+    <origin xyz="-0.015000 0.034000 -0.016000" rpy="-0.000000 -0.000000 -1.570796"/>
     <geometry>
       <mesh filename="file://$(find Robot_description)/meshes/Dynamixel_AX12a__1___7__1.stl" scale="0.001 0.001 0.001"/>
@@ -551,5 +551,5 @@
   </inertial>
   <visual>
-    <origin xyz="-0.046702 -0.041245 -0.148236" rpy="0 0 0"/>
+    <origin xyz="0.015000 -0.034000 -0.016000" rpy="0.000000 0.000000 1.570796"/>
     <geometry>
       <mesh filename="file://$(find Robot_description)/meshes/Dynamixel_AX12a__1___8__1.stl" scale="0.001 0.001 0.001"/>
@@ -558,5 +558,5 @@
   </visual>
   <collision>
-    <origin xyz="-0.046702 -0.041245 -0.148236" rpy="0 0 0"/>
+    <origin xyz="0.015000 -0.034000 -0.016000" rpy="0.000000 0.000000 1.570796"/>
     <geometry>
       <mesh filename="file://$(find Robot_description)/meshes/Dynamixel_AX12a__1___8__1.stl" scale="0.001 0.001 0.001"/>
@@ -571,5 +571,5 @@
   </inertial>
   <visual>
-    <origin xyz="0.046742 -0.002945 -0.148236" rpy="0 0 0"/>
+    <origin xyz="-0.015000 0.034000 -0.016000" rpy="0.000000 -0.000000 -1.570796"/>
     <geometry>
       <mesh filename="file://$(find Robot_description)/meshes/Dynamixel_AX12a__1___3__1.stl" scale="0.001 0.001 0.001"/>
@@ -578,5 +578,5 @@
   </visual>
   <collision>
-    <origin xyz="0.046742 -0.002945 -0.148236" rpy="0 0 0"/>
+    <origin xyz="-0.015000 0.034000 -0.016000" rpy="0.000000 -0.000000 -1.570796"/>
     <geometry>
       <mesh filename="file://$(find Robot_description)/meshes/Dynamixel_AX12a__1___3__1.stl" scale="0.001 0.001 0.001"/>
@@ -591,5 +591,5 @@
   </inertial>
   <visual>
-    <origin xyz="0.114942 -0.040945 -0.148236" rpy="0 0 0"/>
+    <origin xyz="0.015000 -0.034000 -0.016000" rpy="-0.000000 0.000000 1.570796"/>
     <geometry>
       <mesh filename="file://$(find Robot_description)/meshes/Dynamixel_AX12a__1___4__1.stl" scale="0.001 0.001 0.001"/>
@@ -598,5 +598,5 @@
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
Commit message: Update Robot_description package and urdf files

File: Robot_description/urdf/Robot.xacro (robot description, xacro)
@@ -1027,3 +1027,9 @@
   <limit upper="0.698132" lower="-0.698132" effort="100" velocity="100"/>
 </joint>
+<link name="world"/>
+<joint name="fixed_to_world" type="fixed">
+  <parent link="world"/>
+  <child link="base_link"/>
+  <origin xyz="0 0 2" rpy="0 0 0"/>
+</joint>
 </robot>
