Commit message: Phase 2 & 3: Implement Inverse Kinematics and Trot Gait
Changes:
- Added dynamics (damping/friction) and tightened limits for all revolute joints in URDF.
- Added knee linkage plate joints (Revolute 24-27) to ros2_control for full controllability.
- Updated controllers.yaml to include plate joints, set use_sim_time, and enable allow_partial_joints_goal.
- Replaced basic move_dog.py with interactive joint tester (for identifying joint directions).
- Added trot_gait.py script implementing:
  * 2-link planar Inverse Kinematics.
  * Trot gait state machine (diagonal pairs).
  * Body pitch compensation (leaning backward before lifting front legs to prevent forward tipping).
  * Plate joint coupling ratio.

File: Robot_description/urdf/Robot.xacro (robot description, xacro)
@@ -830,4 +830,5 @@
   <axis xyz="0.0 -0.0 -1.0"/>
   <limit upper="0.523599" lower="-0.523599" effort="100" velocity="100"/>
+  <dynamics damping="0.5" friction="0.1"/>
 </joint>
 <joint name="Revolute 14" type="revolute">
@@ -837,4 +838,5 @@
   <axis xyz="-0.0 -0.0 -1.0"/>
   <limit upper="0.523599" lower="-0.523599" effort="100" velocity="100"/>
+  <dynamics damping="0.5" friction="0.1"/>
 </joint>
 <joint name="Revolute 15" type="revolute">
@@ -844,4 +846,5 @@
   <axis xyz="0.0 -0.0 1.0"/>
   <limit upper="0.523599" lower="-0.523599" effort="100" velocity="100"/>
+  <dynamics damping="0.5" friction="0.1"/>
 </joint>
 <joint name="Revolute 16" type="revolute">
@@ -851,28 +854,37 @@
   <axis xyz="0.0 -0.0 1.0"/>
   <limit upper="0.523599" lower="-0.523599" effort="100" velocity="100"/>
-</joint>
-<joint name="Revolute 17" type="continuous">
+  <dynamics damping="0.5" friction="0.1"/>
+</joint>
+<joint name="Revolute 17" type="revolute">
   <origin xyz="0.054898 -0.094919 -0.002" rpy="0 0 0"/>
   <parent link="Robot_Dog_femur__2__1"/>
   <child link="Robot_Dog_TIBIA_1"/>
   <axis xyz="0.0 -0.0 1.0"/>
-</joint>
-<joint name="Revolute 18" type="continuous">
+  <limit lower="-2.356" upper="0.5" effort="100" velocity="100"/>
+  <dynamics damping="0.5" friction="0.1"/>
+</joint>
+<joint name="Revolute 18" type="revolute">
   <origin xyz="0.054898 -0.094919 -0.002" rpy="0 0 0"/>
   <parent link="Robot_Dog_femur__1__1"/>
   <child link="Robot_Dog_TIBIA__1__1"/>
   <axis xyz="0.0 -0.0 1.0"/>
-</joint>
-<joint name="Revolute 21" type="continuous">
+  <limit lower="-2.356" upper="0.5" effort="100" velocity="100"/>
+  <dynamics damping="0.5" friction="0.1"/>
+</joint>
+<joint name="Revolute 21" type="revolute">
   <origin xyz="0.054753 -0.095003 0.002" rpy="0 0 0"/>
   <parent link="Robot_Dog_femur__3__1"/>
   <child link="Robot_Dog_Tibia_Another__1__1"/>
   <axis xyz="-0.0 -0.0 -1.0"/>
-</joint>
-<joint name="Revolute 22" type="continuous">
+  <limit lower="-2.356" upper="0.5" effort="100" velocity="100"/>
+  <dynamics damping="0.5" friction="0.1"/>
+</joint>
+<joint name="Revolute 22" type="revolute">
   <origin xyz="0.054753 -0.095003 0.002" rpy="0 0 0"/>
   <parent link="Robot_Dog_femur_1"/>
   <child link="Robot_Dog_Tibia_Another_1"/>
   <axis xyz="-0.0 -0.0 -1.0"/>
+  <limit lower="-2.356" upper="0.5" effort="100" velocity="100"/>
+  <dynamics damping="0.5" friction="0.1"/>
 </joint>
 <joint name="Revolute 24" type="revolute">
@@ -882,4 +894,5 @@
   <axis xyz="0.0 0.0 1.0"/>
   <limit upper="1.396263" lower="-1.396263" effort="100" velocity="100"/>
+  <dynamics damping="0.5" friction="0.1"/>
 </joint>
 <joint name="Revolute 25" type="revolute">
@@ -889,4 +902,5 @@
   <axis xyz="0.0 -0.0 1.0"/>
   <limit upper="1.396263" lower="-1.396263" effort="100" velocity="100"/>
+  <dynamics damping="0.5" friction="0.1"/>
 </joint>
 <joint name="Revolute 26" type="revolute">
@@ -896,4 +910,5 @@
   <axis xyz="0.0 -0.0 1.0"/>
   <limit upper="1.396263" lower="-1.396263" effort="100" velocity="100"/>
+  <dynamics damping="0.5" friction="0.1"/>
 </joint>
 <joint name="Revolute 27" type="revolute">
@@ -903,4 +918,5 @@
   <axis xyz="0.0 -0.0 -1.0"/>
   <limit upper="1.396263" lower="-1.396263" effort="100" velocity="100"/>
+  <dynamics damping="0.5" friction="0.1"/>
 </joint>
 <joint name="Rigid 28" type="fixed">
@@ -1005,4 +1021,5 @@
   <axis xyz="-1.0 0.0 0.0"/>
   <limit upper="0.698132" lower="-0.698132" effort="100" velocity="100"/>
+  <dynamics damping="0.5" friction="0.1"/>
 </joint>
 <joint name="Revolute 49" type="revolute">
@@ -1012,4 +1029,5 @@
   <axis xyz="-1.0 0.0 0.0"/>
   <limit upper="0.698132" lower="-0.698132" effort="100" velocity="100"/>
+  <dynamics damping="0.5" friction="0.1"/>
 </joint>
 <joint name="Revolute 50" type="revolute">
@@ -1019,4 +1037,5 @@
   <axis xyz="-1.0 0.0 0.0"/>
   <limit upper="0.698132" lower="-0.698132" effort="100" velocity="100"/>
+  <dynamics damping="0.5" friction="0.1"/>
 </joint>
 <joint name="Revolute 51" type="revolute">
@@ -1026,10 +1045,107 @@
   <axis xyz="-1.0 0.0 0.0"/>
   <limit upper="0.698132" lower="-0.698132" effort="100" velocity="100"/>
-</joint>
-<link name="world"/>
-<joint name="fixed_to_world" type="fixed">
-  <parent link="world"/>
-  <child link="base_link"/>
-  <origin xyz="0 0 2" rpy="0 0 0"/>
-</joint>
+  <dynamics damping="0.5" friction="0.1"/>
+</joint>
+<ros2_control name="RobotDogSystem" type="system">
+  <hardware>
+    <plugin>gz_ros2_control/GazeboSimSystem</plugin>
+  </hardware>
+  <!-- Replace the joint names below if they differ from your actual URDF joint names -->
+  <joint name="Revolute 48">
+    <command_interface name="position"><param name="min">-0.698132</param><param name="max">0.698132</param></command_interface>
+    <state_interface name="position"/>
+    <state_interface name="velocity"/>
+    <state_interface name="effort"/>
+  </joint>
+  <joint name="Revolute 49">
+    <command_interface name="position"><param name="min">-0.698132</param><param name="max">0.698132</param></command_interface>
+    <state_interface name="position"/>
+    <state_interface name="velocity"/>
+    <state_interface name="effort"/>
+  </joint>
+  <joint name="Revolute 50">
+    <command_interface name="position"><param name="min">-0.698132</param><param name="max">0.698132</param></command_interface>
+    <state_interface name="position"/>
+    <state_interface name="velocity"/>
+    <state_interface name="effort"/>
+  </joint>
+  <joint name="Revolute 51">
+    <command_interface name="position"><param name="min">-0.698132</param><param name="max">0.698132</param></command_interface>
+    <state_interface name="position"/>
+    <state_interface name="velocity"/>
+    <state_interface name="effort"/>
+  </joint>
+  <joint name="Revolute 13">
+    <command_interface name="position"><param name="min">-0.523599</param><param name="max">0.523599</param></command_interface>
+    <state_interface name="position"/>
+    <state_interface name="velocity"/>
+    <state_interface name="effort"/>
+  </joint>
+  <joint name="Revolute 14">
+    <command_interface name="position"><param name="min">-0.523599</param><param name="max">0.523599</param></command_interface>
+    <state_interface name="position"/>
+    <state_interface name="velocity"/>
+    <state_interface name="effort"/>
+  </joint>
+  <joint name="Revolute 15">
+    <command_interface name="position"><param name="min">-0.523599</param><param name="max">0.523599</param></command_interface>
+    <state_interface name="position"/>
+    <state_interface name="velocity"/>
+    <state_interface name="effort"/>
+  </joint>
+  <joint name="Revolute 16">
+    <command_interface name="position"><param name="min">-0.523599</param><param name="max">0.523599</param></command_interface>
+    <state_interface name="position"/>
+    <state_interface name="velocity"/>
+    <state_interface name="effort"/>
+  </joint>
+  <joint name="Revolute 17">
+    <command_interface name="position"/>
+    <state_interface name="position"/>
+    <state_interface name="velocity"/>
+    <state_interface name="effort"/>
+  </joint>
+  <joint name="Revolute 18">
+    <command_interface name="position"/>
+    <state_interface name="position"/>
+    <state_interface name="velocity"/>
+    <state_interface name="effort"/>
+  </joint>
+  <joint name="Revolute 21">
+    <command_interface name="position"/>
+    <state_interface name="position"/>
+    <state_interface name="velocity"/>
+    <state_interface name="effort"/>
+  </joint>
+  <joint name="Revolute 22">
+    <command_interface name="position"/>
+    <state_interface name="position"/>
+    <state_interface name="velocity"/>
+    <state_interface name="effort"/>
+  </joint>
+  <joint name="Revolute 24">
+    <command_interface name="position"><param name="min">-1.396263</param><param name="max">1.396263</param></command_interface>
+    <state_interface name="position"/>
+    <state_interface name="velocity"/>
+    <state_interface name="effort"/>
+  </joint>
+  <joint name="Revolute 25">
+    <command_interface name="position"><param name="min">-1.396263</param><param name="max">1.396263</param></command_interface>
+    <state_interface name="position"/>
+    <state_interface name="velocity"/>
+    <state_interface name="effort"/>
+  </joint>
+  <joint name="Revolute 26">
+    <command_interface name="position"><param name="min">-1.396263</param><param name="max">1.396263</param></command_interface>
+    <state_interface name="position"/>
+    <state_interface name="velocity"/>
+    <state_interface name="effort"/>
+  </joint>
+  <joint name="Revolute 27">
+    <command_interface name="position"><param name="min">-1.396263</param><param name="max">1.396263</param></command_interface>
+    <state_interface name="position"/>
+    <state_interface name="velocity"/>
+    <state_interface name="effort"/>
+  </joint>
+</ros2_control>
 </robot>
