Commit message: Finalized tuned quadruped motion: bird-leg kinematics, increased URDF effort limits, and ROS sim time state machine sync

File: Robot_description/urdf/Robot.xacro (robot description, xacro)
@@ -7,6 +7,6 @@
   <inertial>
     <origin xyz="1.4662269187703477e-05 0.011546280503874469 -1.4215711144037172e-05" rpy="0 0 0"/>
-    <mass value="0.390197"/>
-    <inertia ixx="0.0006938" iyy="0.0031184" izz="0.0025628" ixy="0" iyz="-0" ixz="4e-07"/>
+    <mass value="0.147350"/>
+    <inertia ixx="0.00026199953" iyy="0.0011776006" izz="0.00096778955" ixy="0" iyz="-0" ixz="1.510519e-07"/>
   </inertial>
   <visual>
@@ -107,6 +107,6 @@
   <inertial>
     <origin xyz="0.022425811828788486 -0.03892583161584007 0.009692501970942596" rpy="0 0 0"/>
-    <mass value="0.033728"/>
-    <inertia ixx="3.42e-05" iyy="1.5e-05" izz="4.48e-05" ixy="1.66e-05" iyz="6e-07" ixz="-4e-07"/>
+    <mass value="0.022710"/>
+    <inertia ixx="2.3027811e-05" iyy="1.0099917e-05" izz="3.0165085e-05" ixy="1.1177241e-05" iyz="4.0399668e-07" ixz="-2.6933112e-07"/>
   </inertial>
   <visual>
@@ -127,6 +127,6 @@
   <inertial>
     <origin xyz="0.022425812909024873 -0.03892583161584007 0.009692502827759242" rpy="0 0 0"/>
-    <mass value="0.033728"/>
-    <inertia ixx="3.42e-05" iyy="1.5e-05" izz="4.48e-05" ixy="1.66e-05" iyz="6e-07" ixz="-4e-07"/>
+    <mass value="0.022710"/>
+    <inertia ixx="2.3027811e-05" iyy="1.0099917e-05" izz="3.0165085e-05" ixy="1.1177241e-05" iyz="4.0399668e-07" ixz="-2.6933112e-07"/>
   </inertial>
   <visual>
@@ -147,6 +147,6 @@
   <inertial>
     <origin xyz="0.022497851507857408 -0.03888423948773731 -0.00969250384848891" rpy="0 0 0"/>
-    <mass value="0.033728"/>
-    <inertia ixx="3.42e-05" iyy="1.5e-05" izz="4.48e-05" ixy="1.66e-05" iyz="-6e-07" ixz="4e-07"/>
+    <mass value="0.022710"/>
+    <inertia ixx="2.3027811e-05" iyy="1.0099917e-05" izz="3.0165085e-05" ixy="1.1177241e-05" iyz="-4.0399668e-07" ixz="2.6933112e-07"/>
   </inertial>
   <visual>
@@ -167,6 +167,6 @@
   <inertial>
     <origin xyz="0.022497852588093767 -0.03888423948773728 -0.009692502991672153" rpy="0 0 0"/>
-    <mass value="0.033728"/>
-    <inertia ixx="3.42e-05" iyy="1.5e-05" izz="4.48e-05" ixy="1.66e-05" iyz="-6e-07" ixz="4e-07"/>
+    <mass value="0.022710"/>
+    <inertia ixx="2.3027811e-05" iyy="1.0099917e-05" izz="3.0165085e-05" ixy="1.1177241e-05" iyz="-4.0399668e-07" ixz="2.6933112e-07"/>
   </inertial>
   <visual>
@@ -187,6 +187,6 @@
   <inertial>
     <origin xyz="-0.02477098826948545 -0.04518985831866687 -0.007607417226580426" rpy="0 0 0"/>
-    <mass value="0.048148"/>
-    <inertia ixx="3.44e-05" iyy="1.38e-05" izz="4.62e-05" ixy="-1.9e-05" iyz="-2e-07" ixz="0"/>
+    <mass value="0.016580"/>
+    <inertia ixx="1.1845809e-05" iyy="4.7520977e-06" izz="1.5909197e-05" ixy="-6.5427432e-06" iyz="-6.8870981e-08" ixz="0"/>
   </inertial>
   <visual>
@@ -207,6 +207,6 @@
   <inertial>
     <origin xyz="-0.024770987189249027 -0.04518985831866685 -0.007607416369763614" rpy="0 0 0"/>
-    <mass value="0.048148"/>
-    <inertia ixx="3.44e-05" iyy="1.38e-05" izz="4.62e-05" ixy="-1.9e-05" iyz="-2e-07" ixz="0"/>
+    <mass value="0.016580"/>
+    <inertia ixx="1.1845809e-05" iyy="4.7520977e-06" izz="1.5909197e-05" ixy="-6.5427432e-06" iyz="-6.8870981e-08" ixz="0"/>
   </inertial>
   <visual>
@@ -227,6 +227,6 @@
   <inertial>
     <origin xyz="-0.024803750749565832 -0.045245780605014954 0.007610469287207489" rpy="0 0 0"/>
-    <mass value="0.048126"/>
-    <inertia ixx="3.44e-05" iyy="1.38e-05" izz="4.62e-05" ixy="-1.9e-05" iyz="2e-07" ixz="-0"/>
+    <mass value="0.016580"/>
+    <inertia ixx="1.1851224e-05" iyy="4.75427e-06" izz="1.5916469e-05" ixy="-6.5457341e-06" iyz="6.8902464e-08" ixz="-0"/>
   </inertial>
   <visual>
@@ -247,6 +247,6 @@
   <inertial>
     <origin xyz="-0.024803749669329522 -0.04524578060501495 0.007610470144024134" rpy="0 0 0"/>
-    <mass value="0.048126"/>
-    <inertia ixx="3.44e-05" iyy="1.38e-05" izz="4.62e-05" ixy="-1.9e-05" iyz="2e-07" ixz="-0"/>
+    <mass value="0.016580"/>
+    <inertia ixx="1.1851224e-05" iyy="4.75427e-06" izz="1.5916469e-05" ixy="-6.5457341e-06" iyz="6.8902464e-08" ixz="-0"/>
   </inertial>
   <visual>
@@ -267,6 +267,6 @@
   <inertial>
     <origin xyz="-0.008503620557143196 -0.009759814247963558 0.004174865661029398" rpy="0 0 0"/>
-    <mass value="0.001815"/>
-    <inertia ixx="0" iyy="0" izz="2e-07" ixy="-0" iyz="0" ixz="0"/>
+    <mass value="0.001200"/>
+    <inertia ixx="0" iyy="0" izz="1.322314e-07" ixy="-0" iyz="0" ixz="0"/>
   </inertial>
   <visual>
@@ -287,6 +287,6 @@
   <inertial>
     <origin xyz="-0.008134902526149346 -0.01006920541177891 -0.0041748658249422255" rpy="0 0 0"/>
-    <mass value="0.001815"/>
-    <inertia ixx="0" iyy="0" izz="2e-07" ixy="-0" iyz="-0" ixz="-0"/>
+    <mass value="0.001200"/>
+    <inertia ixx="0" iyy="0" izz="1.322314e-07" ixy="-0" iyz="-0" ixz="-0"/>
   </inertial>
   <visual>
@@ -307,6 +307,6 @@
   <inertial>
     <origin xyz="-0.008134903606385746 -0.010069205411778939 -0.004174866681759093" rpy="0 0 0"/>
-    <mass value="0.001815"/>
-    <inertia ixx="0" iyy="0" izz="2e-07" ixy="-0" iyz="-0" ixz="-0"/>
+    <mass value="0.001200"/>
+    <inertia ixx="0" iyy="0" izz="1.322314e-07" ixy="-0" iyz="-0" ixz="-0"/>
   </inertial>
   <visual>
@@ -327,6 +327,6 @@
   <inertial>
     <origin xyz="-0.008503621637379555 -0.009759814247963605 0.0041748648042127245" rpy="0 0 0"/>
-    <mass value="0.001815"/>
-    <inertia ixx="0" iyy="0" izz="2e-07" ixy="-0" iyz="0" ixz="0"/>
+    <mass value="0.001200"/>
+    <inertia ixx="0" iyy="0" izz="1.322314e-07" ixy="-0" iyz="0" ixz="0"/>
   </inertial>
   <visual>
@@ -347,6 +347,6 @@
   <inertial>
     <origin xyz="0.0384821258495088 -0.036765030084618525 0.004000437265788498" rpy="0 0 0"/>
-    <mass value="0.014395"/>
-    <inertia ixx="6.2e-06" iyy="6.8e-06" izz="1.28e-05" ixy="6e-06" iyz="-0" ixz="0"/>
+    <mass value="0.017400"/>
+    <inertia ixx="7.4942688e-06" iyy="8.2195207e-06" izz="1.5472039e-05" ixy="7.2525182e-06" iyz="-0" ixz="0"/>
   </inertial>
   <visual>
@@ -367,6 +367,6 @@
   <inertial>
     <origin xyz="0.03848212692974514 -0.03676503008461847 0.004000438122605199" rpy="0 0 0"/>
-    <mass value="0.014395"/>
-    <inertia ixx="6.2e-06" iyy="6.8e-06" izz="1.28e-05" ixy="6e-06" iyz="-0" ixz="0"/>
+    <mass value="0.017400"/>
+    <inertia ixx="7.4942688e-06" iyy="8.2195207e-06" izz="1.5472039e-05" ixy="7.2525182e-06" iyz="-0" ixz="0"/>
   </inertial>
   <visual>
@@ -387,6 +387,6 @@
   <inertial>
     <origin xyz="0.038601163330368726 -0.03664002841539631 -0.004000439143334866" rpy="0 0 0"/>
-    <mass value="0.014395"/>
-    <inertia ixx="6.2e-06" iyy="6.8e-06" izz="1.28e-05" ixy="6e-06" iyz="0" ixz="-0"/>
+    <mass value="0.017400"/>
+    <inertia ixx="7.4942688e-06" iyy="8.2195207e-06" izz="1.5472039e-05" ixy="7.2525182e-06" iyz="0" ixz="-0"/>
   </inertial>
   <visual>
@@ -407,6 +407,6 @@
   <inertial>
     <origin xyz="0.03860116441060513 -0.03664002841539631 -0.004000438286518027" rpy="0 0 0"/>
-    <mass value="0.014395"/>
-    <inertia ixx="6.2e-06" iyy="6.8e-06" izz="1.28e-05" ixy="6e-06" iyz="0" ixz="-0"/>
+    <mass value="0.017400"/>
+    <inertia ixx="7.4942688e-06" iyy="8.2195207e-06" izz="1.5472039e-05" ixy="7.2525182e-06" iyz="0" ixz="-0"/>
   </inertial>
   <visual>
@@ -427,6 +427,6 @@
   <inertial>
     <origin xyz="-0.001783446323468399 -0.0030892144525749843 4.372678115149853e-07" rpy="0 0 0"/>
-    <mass value="0.016680"/>
-    <inertia ixx="1.6e-06" iyy="1.6e-06" izz="1.8e-06" ixy="-0" iyz="0" ixz="0"/>
+    <mass value="0.005860"/>
+    <inertia ixx="5.6211031e-07" iyy="5.6211031e-07" izz="6.323741e-07" ixy="-0" iyz="0" ixz="0"/>
   </inertial>
   <visual>
@@ -447,6 +447,6 @@
   <inertial>
     <origin xyz="-0.0017834452432320264 -0.0030892144525748733 4.3812462796610774e-07" rpy="0 0 0"/>
-    <mass value="0.016680"/>
-    <inertia ixx="1.6e-06" iyy="1.6e-06" izz="1.8e-06" ixy="-0" iyz="-0" ixz="0"/>
+    <mass value="0.005860"/>
+    <inertia ixx="5.6211031e-07" iyy="5.6211031e-07" izz="6.323741e-07" ixy="-0" iyz="-0" ixz="0"/>
   </inertial>
   <visual>
@@ -467,6 +467,6 @@
   <inertial>
     <origin xyz="-0.0017842600017019955 -0.003089391090620397 -4.391453577168303e-07" rpy="0 0 0"/>
-    <mass value="0.016680"/>
-    <inertia ixx="1.6e-06" iyy="1.6e-06" izz="1.8e-06" ixy="-0" iyz="0" ixz="0"/>
+    <mass value="0.005860"/>
+    <inertia ixx="5.6211031e-07" iyy="5.6211031e-07" izz="6.323741e-07" ixy="-0" iyz="0" ixz="0"/>
   </inertial>
   <visual>
@@ -487,6 +487,6 @@
   <inertial>
     <origin xyz="-0.0017842589214655397 -0.0030893910906204247 -4.3828854087712976e-07" rpy="0 0 0"/>
-    <mass value="0.016680"/>
-    <inertia ixx="1.6e-06" iyy="1.6e-06" izz="1.8e-06" ixy="-0" iyz="0" ixz="-0"/>
+    <mass value="0.005860"/>
+    <inertia ixx="5.6211031e-07" iyy="5.6211031e-07" izz="6.323741e-07" ixy="-0" iyz="0" ixz="-0"/>
   </inertial>
   <visual>
@@ -687,6 +687,6 @@
   <inertial>
     <origin xyz="0.02169999879313715 -0.02234992858154677 0.05768838825507094" rpy="0 0 0"/>
-    <mass value="0.070376"/>
-    <inertia ixx="8.54e-05" iyy="0.000103" izz="4.2e-05" ixy="0" iyz="0" ixz="-0"/>
+    <mass value="0.050090"/>
+    <inertia ixx="6.0783307e-05" iyy="7.3310077e-05" izz="2.989343e-05" ixy="0" iyz="0" ixz="-0"/>
   </inertial>
   <visual>
@@ -707,6 +707,6 @@
   <inertial>
     <origin xyz="-0.021700000126626456 -0.02234992858154675 -0.05731161088811228" rpy="0 0 0"/>
-    <mass value="0.070376"/>
-    <inertia ixx="8.54e-05" iyy="0.000103" izz="4.2e-05" ixy="0" iyz="0" ixz="-0"/>
+    <mass value="0.050090"/>
+    <inertia ixx="6.0783307e-05" iyy="7.3310077e-05" izz="2.989343e-05" ixy="0" iyz="0" ixz="-0"/>
   </inertial>
   <visual>
@@ -727,6 +727,6 @@
   <inertial>
     <origin xyz="-0.0003580000073393347 0.012495000006632898 -0.07768476738935479" rpy="0 0 0"/>
-    <mass value="0.068562"/>
-    <inertia ixx="7.46e-05" iyy="9.72e-05" izz="7.84e-05" ixy="8e-07" iyz="0" ixz="-0"/>
+    <mass value="0.046030"/>
+    <inertia ixx="5.0083691e-05" iyy="6.5256498e-05" izz="5.2634871e-05" ixy="5.3709052e-07" iyz="0" ixz="-0"/>
   </inertial>
   <visual>
@@ -747,6 +747,6 @@
   <inertial>
     <origin xyz="0.0014019999998956673 0.01289508354636731 0.07793641610141674" rpy="0 0 0"/>
-    <mass value="0.067804"/>
-    <inertia ixx="7.42e-05" iyy="9.64e-05" izz="7.78e-05" ixy="8e-07" iyz="0" ixz="0"/>
+    <mass value="0.046030"/>
+    <inertia ixx="5.0372043e-05" iyy="6.5442924e-05" izz="5.281597e-05" ixy="5.430948e-07" iyz="0" ixz="0"/>
   </inertial>
   <visual>
@@ -767,6 +767,6 @@
   <inertial>
     <origin xyz="0.00135799891965932 0.012595083546367278 0.07793641524459999" rpy="0 0 0"/>
-    <mass value="0.067804"/>
-    <inertia ixx="7.42e-05" iyy="9.64e-05" izz="7.78e-05" ixy="8e-07" iyz="0" ixz="0"/>
+    <mass value="0.046030"/>
+    <inertia ixx="5.0372043e-05" iyy="6.5442924e-05" izz="5.281597e-05" ixy="5.430948e-07" iyz="0" ixz="0"/>
   </inertial>
   <visual>
@@ -787,6 +787,6 @@
   <inertial>
     <origin xyz="-5.000108757576005e-05 0.012595000006632873 -0.07768476824617163" rpy="0 0 0"/>
-    <mass value="0.068562"/>
-    <inertia ixx="7.46e-05" iyy="9.72e-05" izz="7.84e-05" ixy="8e-07" iyz="0" ixz="-0"/>
+    <mass value="0.046030"/>
+    <inertia ixx="5.0083691e-05" iyy="6.5256498e-05" izz="5.2634871e-05" ixy="5.3709052e-07" iyz="0" ixz="-0"/>
   </inertial>
   <visual>
@@ -829,5 +829,5 @@
   <child link="Robot_Dog_femur__3__1"/>
   <axis xyz="0.0 -0.0 -1.0"/>
-  <limit upper="0.523599" lower="-0.523599" effort="1.5" velocity="6.18"/>
+  <limit upper="2.356" lower="-2.356" effort="25.0" velocity="6.18"/>
   <dynamics damping="0.5" friction="0.1"/>
 </joint>
@@ -837,5 +837,5 @@
   <child link="Robot_Dog_femur_1"/>
   <axis xyz="-0.0 -0.0 -1.0"/>
-  <limit upper="0.523599" lower="-0.523599" effort="1.5" velocity="6.18"/>
+  <limit upper="2.356" lower="-2.356" effort="25.0" velocity="6.18"/>
   <dynamics damping="0.5" friction="0.1"/>
 </joint>
@@ -845,5 +845,5 @@
   <child link="Robot_Dog_femur__2__1"/>
   <axis xyz="0.0 -0.0 1.0"/>
-  <limit upper="0.523599" lower="-0.523599" effort="1.5" velocity="6.18"/>
+  <limit upper="2.356" lower="-2.356" effort="25.0" velocity="6.18"/>
   <dynamics damping="0.5" friction="0.1"/>
 </joint>
@@ -853,5 +853,5 @@
   <child link="Robot_Dog_femur__1__1"/>
   <axis xyz="0.0 -0.0 1.0"/>
-  <limit upper="0.523599" lower="-0.523599" effort="1.5" velocity="6.18"/>
+  <limit upper="2.356" lower="-2.356" effort="25.0" velocity="6.18"/>
   <dynamics damping="0.5" friction="0.1"/>
 </joint>
@@ -861,5 +861,5 @@
   <child link="Robot_Dog_TIBIA_1"/>
   <axis xyz="0.0 -0.0 1.0"/>
-  <limit lower="-2.356" upper="0.5" effort="1.5" velocity="6.18"/>
+  <limit lower="-2.356" upper="2.356" effort="25.0" velocity="6.18"/>
   <dynamics damping="0.5" friction="0.1"/>
 </joint>
@@ -869,5 +869,5 @@
   <child link="Robot_Dog_TIBIA__1__1"/>
   <axis xyz="0.0 -0.0 1.0"/>
-  <limit lower="-2.356" upper="0.5" effort="1.5" velocity="6.18"/>
+  <limit lower="-2.356" upper="2.356" effort="25.0" velocity="6.18"/>
   <dynamics damping="0.5" friction="0.1"/>
 </joint>
@@ -877,5 +877,5 @@
   <child link="Robot_Dog_Tibia_Another__1__1"/>
   <axis xyz="-0.0 -0.0 -1.0"/>
-  <limit lower="-2.356" upper="0.5" effort="1.5" velocity="6.18"/>
+  <limit lower="-2.356" upper="2.356" effort="25.0" velocity="6.18"/>
   <dynamics damping="0.5" friction="0.1"/>
 </joint>
@@ -885,5 +885,5 @@
   <child link="Robot_Dog_Tibia_Another_1"/>
   <axis xyz="-0.0 -0.0 -1.0"/>
-  <limit lower="-2.356" upper="0.5" effort="1.5" velocity="6.18"/>
+  <limit lower="-2.356" upper="2.356" effort="25.0" velocity="6.18"/>
   <dynamics damping="0.5" friction="0.1"/>
 </joint>
@@ -893,5 +893,5 @@
   <child link="Robot_Dog_Knee_Motor_to_Link_Joint__1__1"/>
   <axis xyz="0.0 0.0 1.0"/>
-  <limit upper="1.396263" lower="-1.396263" effort="1.5" velocity="6.18"/>
+  <limit upper="1.396263" lower="-1.396263" effort="25.0" velocity="6.18"/>
   <dynamics damping="0.5" friction="0.1"/>
 </joint>
@@ -901,5 +901,5 @@
   <child link="Robot_Dog_Knee_Motor_to_Link_Joint__2__1"/>
   <axis xyz="0.0 -0.0 1.0"/>
-  <limit upper="1.396263" lower="-1.396263" effort="1.5" velocity="6.18"/>
+  <limit upper="1.396263" lower="-1.396263" effort="25.0" velocity="6.18"/>
   <dynamics damping="0.5" friction="0.1"/>
 </joint>
@@ -909,5 +909,5 @@
   <child link="Robot_Dog_Knee_Motor_to_Link_Joint__3__1"/>
   <axis xyz="0.0 -0.0 1.0"/>
-  <limit upper="1.396263" lower="-1.396263" effort="1.5" velocity="6.18"/>
+  <limit upper="1.396263" lower="-1.396263" effort="25.0" velocity="6.18"/>
   <dynamics damping="0.5" friction="0.1"/>
 </joint>
@@ -917,5 +917,5 @@
   <child link="Robot_Dog_Knee_Motor_to_Link_Joint_1"/>
   <axis xyz="0.0 -0.0 -1.0"/>
-  <limit upper="1.396263" lower="-1.396263" effort="1.5" velocity="6.18"/>
+  <limit upper="1.396263" lower="-1.396263" effort="25.0" velocity="6.18"/>
   <dynamics damping="0.5" friction="0.1"/>
 </joint>
@@ -1049,5 +1049,5 @@
   <child link="Robot_Thigh_and_Tibia_Motor_Right_Box__1__1"/>
   <axis xyz="-1.0 0.0 0.0"/>
-  <limit upper="0.698132" lower="-0.698132" effort="1.5" velocity="6.18"/>
+  <limit upper="0.698132" lower="-0.698132" effort="25.0" velocity="6.18"/>
   <dynamics damping="0.5" friction="0.1"/>
 </joint>
@@ -1057,5 +1057,5 @@
   <child link="Robot_Thigh_and_Tibia_Motor_Left_Box__1__1"/>
   <axis xyz="-1.0 0.0 0.0"/>
-  <limit upper="0.698132" lower="-0.698132" effort="1.5" velocity="6.18"/>
+  <limit upper="0.698132" lower="-0.698132" effort="25.0" velocity="6.18"/>
   <dynamics damping="0.5" friction="0.1"/>
 </joint>
@@ -1065,5 +1065,5 @@
   <child link="Robot_Thigh_and_Tibia_Motor_Left_Box_1"/>
   <axis xyz="-1.0 0.0 0.0"/>
-  <limit upper="0.698132" lower="-0.698132" effort="1.5" velocity="6.18"/>
+  <limit upper="0.698132" lower="-0.698132" effort="25.0" velocity="6.18"/>
   <dynamics damping="0.5" friction="0.1"/>
 </joint>
@@ -1073,5 +1073,5 @@
   <child link="Robot_Thigh_and_Tibia_Motor_Right_Box_1"/>
   <axis xyz="-1.0 0.0 0.0"/>
-  <limit upper="0.698132" lower="-0.698132" effort="1.5" velocity="6.18"/>
+  <limit upper="0.698132" lower="-0.698132" effort="25.0" velocity="6.18"/>
   <dynamics damping="0.5" friction="0.1"/>
 </joint>
@@ -1106,5 +1106,5 @@
   </joint>
   <joint name="Revolute 13">
-    <command_interface name="position"><param name="min">-0.523599</param><param name="max">0.523599</param></command_interface>
+    <command_interface name="position"><param name="min">-2.356</param><param name="max">2.356</param></command_interface>
     <state_interface name="position"/>
     <state_interface name="velocity"/>
@@ -1112,5 +1112,5 @@
   </joint>
   <joint name="Revolute 14">
-    <command_interface name="position"><param name="min">-0.523599</param><param name="max">0.523599</param></command_interface>
+    <command_interface name="position"><param name="min">-2.356</param><param name="max">2.356</param></command_interface>
     <state_interface name="position"/>
     <state_interface name="velocity"/>
@@ -1118,5 +1118,5 @@
   </joint>
   <joint name="Revolute 15">
-    <command_interface name="position"><param name="min">-0.523599</param><param name="max">0.523599</param></command_interface>
+    <command_interface name="position"><param name="min">-2.356</param><param name="max">2.356</param></command_interface>
     <state_interface name="position"/>
     <state_interface name="velocity"/>
@@ -1124,5 +1124,5 @@
   </joint>
   <joint name="Revolute 16">
-    <command_interface name="position"><param name="min">-0.523599</param><param name="max">0.523599</param></command_interface>
+    <command_interface name="position"><param name="min">-2.356</param><param name="max">2.356</param></command_interface>
     <state_interface name="position"/>
     <state_interface name="velocity"/>
